File: PCB/schema_electrica/schema_electrica.kicad_sch (KiCad schematic)
At the start: 17 parts

Commit message: final-update
Parts:
- added R?: 470, symbol Device:R
- R?: value R -> 250
Connections:
- net GND: no longer D?.1 (K)
- net VCC: now also D?.1 (K)
- net at D?.2 (A): now also R?.2; no longer U?.20 (PD6)
- new net: R?.1, U?.20 (PD6)
Other:
- moved on the sheet: 22pF, 7.32Mhz, BZ?, C?, D?, J?, LD?, R?, SW?, U?
